Commit message: robots, namespaced, together in rviz and gz w moveit

File: nemo1_description/urdf/nemo1.urdf (robot description, URDF)
Before this commit: robot nemo1, 9 links, 8 joints
Joints:
- joint fixedFrameToWorld: origin xyz=88.8 -0.6 -35.2 rpy=0.0 0.0 0.0 -> xyz=89.8 -0.6 -35.2 rpy=0.0 0.0 0.0
