Commit message: namespaced both robots individually

File: bean2_moveit/config/bean2.urdf.xacro (robot description, xacro)
@@ -11,5 +11,8 @@
     <gazebo>
 	    <plugin filename="gz_ros2_control-system"
-	    name="gz_ros2_control::GazeboSimROS2ControlPlugin">
+		    name="gz_ros2_control::GazeboSimROS2ControlPlugin">
+	    <ros>
+		    <namespace>bean</namespace>
+	    </ros>
 	    <parameters>$(find bean2_moveit)/config/ros2_controllers.yaml</parameters>
 	    </plugin>

File: bean3_description/urdf/bean2.urdf (robot description, URDF)
Before this commit: robot bean2, 8 links, 7 joints
Links:
- removed link base_link
- added link bean_base_link, mass 140.69; collision mesh filename=package://bean3_description/meshes/base_link.STL; visual mesh filename=package://bean3_description/meshes/base_link.STL
Joints:
- joint fixedFrameToWorld: child base_link -> bean_base_link
- joint joint_one: parent base_link -> bean_base_link

File: nemo1_description/urdf/nemo1.urdf (robot description, URDF)
Before this commit: robot nemo1, 9 links, 8 joints
Links:
- removed link base_link
- added link nemo_base_link, mass 39.819; collision mesh filename=package://nemo1_description/meshes/base_link.STL; visual mesh filename=package://nemo1_description/meshes/base_link.STL
Joints:
- joint J1: parent base_link -> nemo_base_link
- joint fixedFrameToWorld: child base_link -> nemo_base_link

File: nemo1_moveit/config/nemo1.urdf.xacro (robot description, xacro)
@@ -12,4 +12,7 @@
 	    <plugin filename="gz_ros2_control-system"
 		    name="gz_ros2_control::GazeboSimROS2ControlPlugin">
+		    <ros>
+			    <namespace>nemo</namespace>
+		    </ros>
 		    <parameters>$(find nemo1_moveit)/config/ros2_controllers.yaml</parameters>
 	    </plugin>

Commit message: typos

File: bean2_moveit/config/bean2.urdf.xacro (robot description, xacro)
@@ -16,4 +16,5 @@
 	    </ros>
 	    <parameters>$(find bean2_moveit)/config/ros2_controllers.yaml</parameters>
+    </plugin>
     <!-- detachable joint plugin -->
 	    <plugin filename="gz-sim-detachable-joint-system"

File: bean3_description/urdf/bean2.urdf (robot description, URDF)
Before this commit: robot bean2, 9 links, 8 joints
Joints:
- removed joint docking_frame
- added joint docking_joint: type fixed, parent link_six, child docking_frame, origin xyz=0.0 0.0 -0.333 rpy=0.0 0.0 0.0
