Commit message: spawned robots at correct ISS coordinates

File: bean3_description/urdf/bean2.urdf (robot description, URDF)
Before this commit: robot bean2, 8 links, 7 joints
Joints:
- joint fixedFrameToWorld: origin xyz=0.0 0.0 0.0 rpy=0.0 0.0 0.0 -> xyz=92.6 -2.35 -35 rpy=1.57 1.57 0.0

File: nemo1_description/urdf/nemo1.urdf (robot description, URDF)
Before this commit: robot nemo1, 8 links, 7 joints
Links:
- added link world
Joints:
- added joint fixedFrameToWorld: type fixed, parent world, child base_link, origin xyz=88.8 -0.6 -35.2 rpy=0.0 0.0 0.0

Commit message: more model updates for sim task

File: bean3_description/urdf/bean2.urdf (robot description, URDF)
Before this commit: robot bean2, 8 links, 7 joints
Links:
- added link docking_frame, mass 0.001; collision sphere radius=0.005; visual sphere radius=0.005
Joints:
- added joint docking_frame: type fixed, parent link_six, child docking_link, origin xyz=0.0 0.0 -0.333 rpy=0.0 0.0 0.0

Commit message: new bean and capsule spawn location

File: bean3_description/urdf/bean2.urdf (robot description, URDF)
Before this commit: robot bean2, 9 links, 8 joints
Joints:
- joint fixedFrameToWorld: origin xyz=92.6 -2.35 -35 rpy=1.57 1.57 0.0 -> xyz=90.1 -1.95 -36.0 rpy=1.57 1.57 0.0
